File: SillyTinySCSI.kicad_sch (KiCad schematic)
At the start: 24 parts, among them J302 DB25_Plug, U101 74LVT125, U102 74LVT125, U105 74LVT245, U106 74LVT245

Commit message: fix BOM and proposed RTM files
Parts:
- J302: LCSC (none) -> D25P24B4PA00LF; Manufacturer (none) -> Amphenol ICC (FCI); PN D25P24B4PA00LF -> (none); PartNumber (none) -> D25P24B4PA00LF; digikey (none) -> 609-5556-ND
- RN301, RN302: value 110 -> 120; LCSC (none) -> C1731305; Manufacturer (none) -> Panasonic; PartNumber (none) -> EXB-2HV121JV; digikey (none) -> Y1121CT-ND
Changed lines of the file:
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@@
       (effects (font (size 1.27 1.27)))
     )
-    (property "Value" "110" (at 257.81 82.55 90)
+    (property "Value" "120" (at 257.81 82.55 90)
       (effects (font (size 1.27 1.27)))
     )
@@
     )
     (property "Datasheet" "~" (at 257.81 93.98 0)
+      (effects (font (size 1.27 1.27)) hide)
+    )
+    (property "LCSC" "C1731305" (at 257.81 93.98 90)
+      (effects (font (size 1.524 1.524)) hide)
+    )
+    (property "P/N" "" (at 257.81 93.98 90)
+      (effects (font (size 1.524 1.524)) hide)
+    )
+    (property "PartNumber" "EXB-2HV121JV" (at 257.81 93.98 0)
+      (effects (font (size 1.27 1.27)) hide)
+    )
+    (property "Manufacturer" "Panasonic" (at 257.81 93.98 0)
+      (effects (font (size 1.27 1.27)) hide)
+    )
+    (property "digikey" "Y1121CT-ND" (at 257.81 93.98 0)
       (effects (font (size 1.27 1.27)) hide)
     )
@@
       (effects (font (size 1.27 1.27)))
     )
-    (property "Value" "110" (at 257.81 31.75 90)
+    (property "Value" "120" (at 257.81 31.75 90)
       (effects (font (size 1.27 1.27)))
     )
@@
     )
     (property "Datasheet" "~" (at 257.81 43.18 0)
+      (effects (font (size 1.27 1.27)) hide)
+    )
+    (property "LCSC" "C1731305" (at 257.81 43.18 90)
+      (effects (font (size 1.524 1.524)) hide)
+    )
+    (property "P/N" "" (at 257.81 43.18 90)
+      (effects (font (size 1.524 1.524)) hide)
+    )
+    (property "PartNumber" "EXB-2HV121JV" (at 257.81 43.18 0)
+      (effects (font (size 1.27 1.27)) hide)
+    )
+    (property "Manufacturer" "Panasonic" (at 257.81 43.18 0)
+      (effects (font (size 1.27 1.27)) hide)
+    )
+    (property "digikey" "Y1121CT-ND" (at 257.81 43.18 0)
       (effects (font (size 1.27 1.27)) hide)
     )
@@
       (effects (font (size 1.27 1.27)) hide)
     )
-    (property "PN" "D25P24B4PA00LF" (at 30.48 187.96 0)
+    (property "PN" "" (at 30.48 187.96 0)
       (effects (font (size 1.524 1.524)))
     )
+    (property "PartNumber" "D25P24B4PA00LF" (at 30.48 151.13 0)
+      (effects (font (size 1.27 1.27)) hide)
+    )
+    (property "LCSC" "D25P24B4PA00LF" (at 30.48 151.13 0)
+      (effects (font (size 1.27 1.27)) hide)
+    )
+    (property "Manufacturer" "Amphenol ICC (FCI)" (at 30.48 151.13 0)
+      (effects (font (size 1.27 1.27)) hide)
+    )
+    (property "digikey" "609-5556-ND" (at 30.48 151.13 0)
+      (effects (font (size 1.27 1.27)) hide)
+    )
     (pin "1")
