File: cpu.kicad_sch (KiCad schematic)
At the start: 17 parts, among them J301 Micro_SD_Card_Det1, U1 Pico W

Commit message: fix BOM and proposed RTM files
Parts:
- added D304: LED, LED_SMD:LED_0805_2012Metric, symbol zuluscsi-rescue:LED
- D302: JLCPCB_IGNORE (none) -> do not fit; LCSC C434435 -> n/a; PartNumber LY R976-PS-36 -> HSMC-C170-T0000; digikey 475-2560-1-ND -> 516-HSMC-C170-T0000CT-ND
- J301: LCSC (none) -> n/a; Manufacturer (none) -> Molex; PartNumber (none) -> 1051620001; digikey (none) -> WM14405CT-ND
- R304: value 62 -> 51; LCSC C25252 -> C23197; PartNumber RC0603FR-0762RL -> 0603WAF510JT5E; digikey 311-62.0HRTR-ND -> (none)
Connections:
- net GND: now also D304.1 (K)
- net at D302.2 (A), R304.1: now also D304.2 (A)
Other:
- moved on the sheet: D302
Changed lines of the file:
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@@
   (junction (at 234.95 34.29) (diameter 0) (color 0 0 0 0)
   )
+  (junction (at 82.55 139.7) (diameter 0) (color 0 0 0 0)
+  )
   (junction (at 99.06 58.42) (diameter 0) (color 0 0 0 0)
   )
@@
   )
   (junction (at 201.93 105.41) (diameter 0) (color 0 0 0 0)
+  )
+  (junction (at 82.55 129.54) (diameter 0) (color 0 0 0 0)
   )
   (junction (at 201.93 133.35) (diameter 0) (color 0 0 0 0)
@@
     (stroke (width 0) (type default))
   )
+  (wire (pts (xy 82.55 139.7) (xy 82.55 138.43))
+    (stroke (width 0) (type default))
+  )
+  (wire (pts (xy 82.55 130.81) (xy 82.55 129.54))
+    (stroke (width 0) (type default))
+  )
   (wire (pts (xy 99.06 58.42) (xy 99.06 71.12))
     (stroke (width 0) (type default))
@@
     (stroke (width 0) (type default))
   )
+  (wire (pts (xy 92.71 129.54) (xy 82.55 129.54))
+    (stroke (width 0) (type default))
+  )
   (wire (pts (xy 168.91 120.65) (xy 171.45 120.65))
     (stroke (width 0) (type default))
@@
     (stroke (width 0) (type default))
   )
+  (wire (pts (xy 92.71 139.7) (xy 82.55 139.7))
+    (stroke (width 0) (type default))
+  )
   (wire (pts (xy 256.54 63.5) (xy 261.62 63.5))
     (stroke (width 0) (type default))
@@
     (stroke (width 0) (type default))
   )
+  (wire (pts (xy 82.55 142.24) (xy 82.55 139.7))
+    (stroke (width 0) (type default))
+  )
   (wire (pts (xy 191.77 102.87) (xy 196.85 102.87))
     (stroke (width 0) (type default))
@@
     (stroke (width 0) (type default))
   )
+  (wire (pts (xy 92.71 129.54) (xy 92.71 130.81))
+    (stroke (width 0) (type default))
+  )
   (wire (pts (xy 99.06 33.02) (xy 99.06 45.72))
     (stroke (width 0) (type default))
@@
   )
   (wire (pts (xy 168.91 135.89) (xy 186.69 135.89))
+    (stroke (width 0) (type default))
+  )
+  (wire (pts (xy 92.71 138.43) (xy 92.71 139.7))
     (stroke (width 0) (type default))
   )
@@
     )
   )
-  (symbol (lib_id "zuluscsi-rescue:LED") (at 82.55 133.35 90) (unit 1)
-    (in_bom yes) (on_board yes) (dnp no)
-    (property "Reference" "D302" (at 85.5472 132.3594 90)
+  (symbol (lib_id "zuluscsi-rescue:LED") (at 82.55 134.62 90) (unit 1)
+    (in_bom yes) (on_board yes) (dnp no)
+    (property "Reference" "D302" (at 85.5472 133.6294 90)
       (effects (font (size 1.27 1.27)) (justify right))
     )
-    (property "Value" "LED" (at 85.5472 134.6708 90)
+    (property "Value" "LED" (at 85.5472 135.9408 90)
       (effects (font (size 1.27 1.27)) (justify right))
     )
-    (property "Footprint" "LED_SMD:LED_0805_2012Metric" (at 82.55 133.35 0)
-      (effects (font (size 1.27 1.27)) hide)
-    )
-    (property "Datasheet" "" (at 82.55 133.35 0)
-      (effects (font (size 1.27 1.27)))
-    )
-    (property "LCSC" "C434435" (at 82.55 133.35 0)
-      (effects (font (size 1.27 1.27)) hide)
-    )
-    (property "Manufacturer" "Osram Opto Semiconductors Inc" (at 82.55 133.35 0)
-      (effects (font (size 1.27 1.27)) hide)
-    )
-    (property "PartNumber" "LY R976-PS-36" (at 82.55 133.35 0)
-      (effects (font (size 1.27 1.27)) hide)
-    )
-    (property "digikey" "475-2560-1-ND" (at 82.55 133.35 0)
-      (effects (font (size 1.27 1.27)) hide)
-    )
-    (property "JLCPCBCORRECT" "" (at 82.55 133.35 0)
-      (effects (font (size 1.27 1.27)) hide)
-    )
-    (property "JLCPCB_IGNORE" "" (at 82.55 133.35 0)
+    (property "Footprint" "LED_SMD:LED_0805_2012Metric" (at 82.55 134.62 0)
+      (effects (font (size 1.27 1.27)) hide)
+    )
+    (property "Datasheet" "" (at 82.55 134.62 0)
+      (effects (font (size 1.27 1.27)))
+    )
+    (property "LCSC" "n/a" (at 82.55 134.62 0)
+      (effects (font (size 1.27 1.27)) hide)
+    )
+    (property "Manufacturer" "Osram Opto Semiconductors Inc" (at 82.55 134.62 0)
+      (effects (font (size 1.27 1.27)) hide)
+    )
+    (property "PartNumber" "HSMC-C170-T0000" (at 82.55 134.62 0)
+      (effects (font (size 1.27 1.27)) hide)
+    )
+    (property "digikey" "516-HSMC-C170-T0000CT-ND" (at 82.55 134.62 0)
+      (effects (font (size 1.27 1.27)) hide)
+    )
+    (property "JLCPCBCORRECT" "" (at 82.55 134.62 0)
+      (effects (font (size 1.27 1.27)) hide)
+    )
+    (property "JLCPCB_IGNORE" "do not fit" (at 82.55 134.62 0)
       (effects (font (size 1.27 1.27)) hide)
     )
@@
       (effects (font (size 1.27 1.27)) (justify right))
     )
-    (property "Value" "62" (at 84.328 126.873 0)
+    (property "Value" "51" (at 84.328 126.873 0)
       (effects (font (size 1.27 1.27)) (justify right))
     )
@@
       (effects (font (size 1.27 1.27)))
     )
-    (property "LCSC" "C25252" (at 82.55 125.73 0)
+    (property "LCSC" "C23197" (at 82.55 125.73 0)
       (effects (font (size 1.27 1.27)) hide)
     )
@@
       (effects (font (size 1.27 1.27)) hide)
     )
-    (property "PartNumber" "RC0603FR-0762RL" (at 82.55 125.73 0)
-      (effects (font (size 1.27 1.27)) hide)
-    )
-    (property "digikey" "311-62.0HRTR-ND" (at 82.55 125.73 0)
+    (property "PartNumber" "0603WAF510JT5E" (at 82.55 125.73 0)
+      (effects (font (size 1.27 1.27)) hide)
+    )
+    (property "digikey" "" (at 82.55 125.73 0)
       (effects (font (size 1.27 1.27)) hide)
     )
@@
     )
   )
-  (symbol (lib_id "zuluscsi-rescue:GND") (at 82.55 137.16 0) (mirror y) (unit 1)
-    (in_bom yes) (on_board yes) (dnp no)
-    (property "Reference" "#PWR0314" (at 82.55 143.51 0)
-      (effects (font (size 1.27 1.27)) hide)
-    )
-    (property "Value" "GND" (at 82.55 140.97 0)
-      (effects (font (size 1.27 1.27)))
-    )
-    (property "Footprint" "" (at 82.55 137.16 0)
-      (effects (font (size 1.27 1.27)))
-    )
-    (property "Datasheet" "" (at 82.55 137.16 0)
+  (symbol (lib_id "zuluscsi-rescue:GND") (at 82.55 142.24 0) (unit 1)
+    (in_bom yes) (on_board yes) (dnp no)
+    (property "Reference" "#PWR0314" (at 82.55 148.59 0)
+      (effects (font (size 1.27 1.27)) hide)
+    )
+    (property "Value" "GND" (at 82.55 146.05 0)
+      (effects (font (size 1.27 1.27)))
+    )
+    (property "Footprint" "" (at 82.55 142.24 0)
+      (effects (font (size 1.27 1.27)))
+    )
+    (property "Datasheet" "" (at 82.55 142.24 0)
       (effects (font (size 1.27 1.27)))
     )
@@
     )
   )
+  (symbol (lib_id "zuluscsi-rescue:LED") (at 92.71 134.62 90) (unit 1)
+    (in_bom yes) (on_board yes) (dnp no)
+    (property "Reference" "D304" (at 95.7072 133.6294 90)
+      (effects (font (size 1.27 1.27)) (justify right))
+    )
+    (property "Value" "LED" (at 95.7072 135.9408 90)
+      (effects (font (size 1.27 1.27)) (justify right))
+    )
+    (property "Footprint" "LED_SMD:LED_0805_2012Metric" (at 92.71 134.62 0)
+      (effects (font (size 1.27 1.27)) hide)
+    )
+    (property "Datasheet" "" (at 92.71 134.62 0)
+      (effects (font (size 1.27 1.27)))
+    )
+    (property "LCSC" "n/a" (at 92.71 134.62 0)
+      (effects (font (size 1.27 1.27)) hide)
+    )
+    (property "Manufacturer" "Osram Opto Semiconductors Inc" (at 92.71 134.62 0)
+      (effects (font (size 1.27 1.27)) hide)
+    )
+    (property "PartNumber" "HSMC-C170-T0000" (at 92.71 134.62 0)
+      (effects (font (size 1.27 1.27)) hide)
+    )
+    (property "digikey" "516-HSMC-C170-T0000CT-ND" (at 92.71 134.62 0)
+      (effects (font (size 1.27 1.27)) hide)
+    )
+    (property "JLCPCBCORRECT" "" (at 92.71 134.62 0)
+      (effects (font (size 1.27 1.27)) hide)
+    )
+    (property "JLCPCB_IGNORE" "do not fit" (at 92.71 134.62 0)
+      (effects (font (size 1.27 1.27)) hide)
+    )
+    (pin "1")
+    (pin "2")
+    (instances
+      (project "SillyTinySCSI"
+        (path "/0a1a4d88-972a-46ce-b25e-6cb796bd41f7/00000000-0000-0000-0000-000055ff7cc4"
+          (reference "D304") (unit 1)
+        )
+      )
+    )
+  )
   (symbol (lib_id "zuluscsi-rescue:+3V0") (at 233.68 34.29 90) (mirror x) (unit 1)
     (in_bom yes) (on_board yes) (dnp no)
@@
       (effects (font (size 1.27 1.27)) hide)
     )
-    (property "Datasheet" "https://datasheet.lcsc.com/lcsc/2110151630_XKB-Connectivity-XKTF-015-N_C381082.pdf" (at 233.68 128.27 0)
-      (effects (font (size 1.27 1.27)) hide)
-    )
+    (property "Datasheet" "" (at 233.68 128.27 0)
+      (effects (font (size 1.27 1.27)) hide)
+    )
+    (property "LCSC" "n/a" (at 233.68 130.81 0)
+      (effects (font (size 1.524 1.524)) hide)
+    )
+    (property "Manufacturer" "Molex" (at 233.68 130.81 0)
+      (effects (font (size 1.27 1.27)) hide)
+    )
+    (property "PartNumber" "1051620001" (at 233.68 130.81 0)
+      (effects (font (size 1.27 1.27)) hide)
+    )
+    (property "digikey" "WM14405CT-ND" (at 233.68 130.81 0)
+      (effects (font (size 1.27 1.27)) hide)
+    )
