File: V2.0/SillyTinySCSI.kicad_pcb (KiCad board)
At the start: 4 copper layers, 53.5 x 25 mm, 62 parts, among them J1 DB25_Plug, J2 Micro_SD_Card_Det1, U1 74LVT125, U2 74LVT245, U3 74LVT125, U4 74LVT245, U5 TLV75728PDBVR, U6 Pico W

Commit message: rearrange
Parts:
- moved U1 21.4 mm to (144.0, 72.2)
- moved R17 18.6 mm to (128.0, 57.7), turned to 0 degrees
- moved R14 18.4 mm to (145.7, 56.0), turned to 0 degrees
- moved R27 18.4 mm to (119.7, 73.1), turned to -90 degrees
- moved R29 16.9 mm to (121.3, 68.8), turned to -90 degrees
- moved C1 16.2 mm to (142.5, 51.2), turned to 0 degrees
- moved R7 15.3 mm to (145.4, 67.8), turned to 0 degrees
- moved R25 15.2 mm to (122.9, 73.1), turned to -90 degrees
- moved R22 15.1 mm to (142.6, 56.0), turned to 0 degrees
- moved R28 14.9 mm to (119.7, 68.8), turned to 90 degrees
- moved R1 14.7 mm to (142.4, 67.8), turned to 0 degrees
- moved R6 14.1 mm to (118.1, 73.1), turned to 90 degrees
- moved R31 13.6 mm to (124.5, 68.8), turned to -90 degrees
- moved U4 13.5 mm to (130.9, 71.2)
- moved R26 13.2 mm to (121.3, 73.1), turned to -90 degrees
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Routing:
- net +2V8: track 41.0 -> 58.7 mm
- net ~{DATA_DIR}: track 0.00 -> 10.1 mm
- net ~{SCSI_DB3}: track 0.00 -> 8.29 mm
- net ~{SCSI_DB4}: track 0.00 -> 8.21 mm
- net ~{SCSI_DB2}: track 0.00 -> 6.75 mm
- net ~{SCSI_DB5}: track 12.9 -> 7.02 mm
- net ~{SCSI_DB6}: track 0.00 -> 5.15 mm
- net ~{SCSI_DB0}: track 0.00 -> 3.39 mm
- net ~{SCSI_DB7}: track 0.00 -> 3.28 mm
- net ~{SCSI_DB1}: track 8.17 -> 5.21 mm
- net GND: vias 3 -> 5

Commit message: pwr routed
Parts:
- removed L2: Ferrite_Bead_Small, Inductor_SMD:L_0603_1608Metric
- D1, D2: footprint Diode_SMD:D_SOD-123 -> Diode_SMD:D_SOD-323
- moved F1 13.8 mm to (110.8, 55.8), turned to 0 degrees
- moved D1 12.5 mm to (117.0, 68.0)
- moved L1 10.6 mm to (110.6, 57.8), turned to 180 degrees
- moved C10 7.46 mm to (121.6, 55.5)
- moved C7 7.41 mm to (121.6, 57.5)
- moved D2 5.26 mm to (118.6, 56.4), turned to 90 degrees
- moved U5 5.00 mm to (115.5, 56.3)
- moved C13 3.60 mm to (113.6, 69.8), turned to 180 degrees
- moved C12 1.85 mm to (113.6, 68.0), turned to 180 degrees
- moved C15 1.78 mm to (125.6, 54.0), turned to -90 degrees
- moved R16 0.57 mm to (110.2, 68.0)
- moved C14 0.45 mm to (137.9, 72.2)
- moved U2 0.38 mm to (135.5, 54.7)
- moved R10 0.36 mm to (128.3, 54.6)
- moved R11 0.36 mm to (128.3, 53.0)
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Connections:
- C7 pad 1: +5V -> /power/5V_REG
- C8 pad 1: +5V -> /power/5V_REG
- C9 pad 1: +5V -> +2V8
- D1 pad 1: /power/5V_IN -> 5V_IN
- D2 pad 1: +5V -> /power/5V_REG
- F1 pad 2: +5V -> /power/5V_REG
- L1 pad 2: /power/5V_IN -> 5V_IN
- U5 pad 1: +5V -> /power/5V_REG
- U5 pad 3: +5V -> /power/5V_REG
- U6 pad 39: Net-(U6-VSYS) -> 5V_IN
Routing:
- net +5V: track 50.3 -> 0.00 mm, vias 2 -> 0
- net 5V_IN: track 0.00 -> 24.8 mm, vias 0 -> 1
- net /power/5V_REG: track 0.00 -> 17.6 mm
- net /power/5V_IN: track 13.2 -> 0.00 mm, vias 2 -> 0
- net Net-(U6-VSYS): track 12.3 -> 0.00 mm, vias 1 -> 0
- net GND: track 41.9 -> 36.5 mm
- net TERMPWR_5V: track 9.60 -> 4.55 mm, vias 1 -> 0
- net +2V8: track 58.7 -> 63.2 mm
- net ~{GPIO_DB2}: track 2.46 -> 0.00 mm
- net ~{GPIO_DB1}: track 1.39 -> 0.00 mm

Commit message: routing and drc 1
Parts:
- moved R13 0.20 mm to (153.0, 68.2)
- turned C2 to 180 degrees
Routing:
- net +2V8: track 63.2 -> 251.6 mm, vias 2 -> 7
- net GND: track 36.5 -> 132.7 mm, vias 5 -> 24
- net /cpu/SDIO_D0: track 0.00 -> 63.6 mm, vias 0 -> 2
- net /cpu/SDIO_D3: track 0.00 -> 62.6 mm, vias 0 -> 2
- net /cpu/SDIO_D2: track 0.00 -> 59.3 mm, vias 0 -> 1
- net /cpu/SDIO_D1: track 0.00 -> 59.3 mm, vias 0 -> 1
- net /cpu/SDIO_CMD: track 0.00 -> 44.9 mm, vias 0 -> 2
- net /cpu/SDIO_CLK: track 0.00 -> 43.4 mm
- net ~{DATA_DIR}: track 10.1 -> 48.4 mm, vias 0 -> 3
- net ~{SCSI_DBP}: track 0.00 -> 37.9 mm, vias 0 -> 2
- net ~{DBGLOG}: track 0.00 -> 30.5 mm, vias 0 -> 2
- net ~{OUT_BSY}: track 0.00 -> 29.8 mm, vias 0 -> 3
- net ~{IN_RST}: track 0.00 -> 29.4 mm, vias 0 -> 2
- net ~{GPIO_DBP}: track 0.00 -> 28.6 mm, vias 0 -> 2
- net ~{SCSI_REQ}: track 0.00 -> 27.7 mm, vias 0 -> 1
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
Commit message: sync up
Parts:
- removed RN3: 4k7, Resistor_SMD:R_Array_Convex_4x0603
- added R32: 4k7, Resistor_SMD:R_0603_1608Metric, B.Cu at (160.7, 69.7)
- added R33: 4k7, Resistor_SMD:R_0603_1608Metric, B.Cu at (159.2, 69.7)
- added R34: 4k7, Resistor_SMD:R_0603_1608Metric, B.Cu at (157.7, 69.7)
- added R35: 4k7, Resistor_SMD:R_0603_1608Metric, B.Cu at (156.2, 69.7)
- L1: footprint Inductor_SMD:L_0603_1608Metric -> Inductor_SMD:L_0805_2012Metric
- moved C4 0.90 mm to (154.7, 69.7)
- moved C3 0.80 mm to (152.2, 70.2), turned to 0 degrees
- moved R13 0.70 mm to (152.3, 68.2)
- moved F1 0.16 mm to (110.6, 55.7), turned to 180 degrees
- moved R18 0.14 mm to (159.3, 56.8)
- moved C6 0.14 mm to (158.5, 54.4)
- moved R15 0.14 mm to (160.1, 54.4)
- moved L1 0.10 mm to (110.7, 57.8)
- turned C9 to 180 degrees
Connections:
- D1 pad 1: 5V_IN -> Net-(D1-K)
- F1 pad 1: Net-(F1-Pad1) -> Net-(D1-K)
- F1 pad 2: /power/5V_REG -> +5VP
- L1 pad 1: Net-(F1-Pad1) -> /power/5V_REG
- L1 pad 2: 5V_IN -> +5VP
- U6 pad 39: 5V_IN -> +5VP
Routing:
- net +2V8: track 251.6 -> 280.4 mm, vias 7 -> 9
- net 5V_IN: track 23.0 -> 0.00 mm, vias 1 -> 0
- net Net-(D1-K): track 0.00 -> 15.2 mm
- net +5VP: track 0.00 -> 12.4 mm, vias 0 -> 1
- net ~{GPIO_DB5}: track 16.5 -> 11.7 mm
- net ~{GPIO_ACK}: track 12.8 -> 9.11 mm
- net Net-(F1-Pad1): track 3.43 -> 0.00 mm
- net /power/5V_REG: track 17.1 -> 20.5 mm
- net /cpu/SDIO_D2: track 59.3 -> 56.6 mm
- net ~{GPIO_MSG_BSY}: track 24.8 -> 22.2 mm
- net /cpu/SDIO_CLK: track 43.4 -> 41.3 mm
- net ~{GPIO_DB2}: track 20.4 -> 18.5 mm
- net ~{GPIO_ATN}: track 9.84 -> 8.07 mm
- net GND: track 132.7 -> 134.3 mm, vias 24 -> 25
- net ~{GPIO_DB4}: track 14.6 -> 13.2 mm
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
Commit message: vers
Routing:
- net GND: track 134.3 -> 137.6 mm, vias 25 -> 26
Other:
- board text added: "< Pico USB<"

Commit message: bring current
Parts:
- added R36: 4k7, Resistor_SMD:R_0603_1608Metric, B.Cu at (145.7, 57.8)
Connections:
- R15 pad 2: /cpu/LED_SWO -> Net-(R15-Pad2)
- U1 pad 8: unconnected-(U1-Pad8) -> Net-(R15-Pad2)
- U1 pad 9: GND -> /cpu/LED_SWO
- U6 pad 27: ~{IN_RST} -> Net-(U6-GPIO21)
Routing:
- net Net-(R15-Pad2): track 0.00 -> 32.3 mm, vias 0 -> 2
- net /cpu/LED_SWO: track 2.62 -> 34.5 mm, vias 1 -> 2
- net Net-(U6-GPIO21): track 0.00 -> 12.2 mm, vias 0 -> 2
- net +2V8: track 280.6 -> 292.4 mm, vias 9 -> 10
- net ~{IN_RST}: track 29.4 -> 20.5 mm
- net +5VP: track 12.4 -> 11.3 mm
- net ~{DATA_DIR}: track 47.2 -> 46.4 mm
- net ~{DBGLOG}: track 30.1 -> 29.3 mm
- net ~{GPIO_DBP}: track 28.3 -> 28.9 mm
- net GND: track 137.6 -> 138.0 mm, vias 26 -> 25

Commit message: bring current
Parts:
- turned C6 to 90 degrees
Connections:
- U2 pad 3: GND -> unconnected-(U2-A1-Pad3)
- U2 pad 9: GND -> unconnected-(U2-A7-Pad9)
Routing:
- net GND: track 138.0 -> 159.8 mm, vias 25 -> 24
- net +2V8: track 292.4 -> 299.0 mm
- net ~{DBGLOG}: track 29.3 -> 28.0 mm
- net ~{SCSI_BSY}: track 26.6 -> 27.3 mm
