File: V2.0/SillyTinySCSI.kicad_sch (KiCad schematic)
At the start: 38 parts, among them J1 DB25_Plug, U1 74LVT125, U2 74LVT245, U3 74LVT125, U4 74LVT245

Commit message: bring current
Connections:
- net GND: no longer U2.3 (A1), U2.9 (A7)
- no-connect marks 2 -> 4
Other:
- note added: "/RST is input only in target mode. /RST is bidirectional by definition, but zuluscsi will not drive it in target mode, only as an initiator."
- note removed: "RST is input only in target mode. it is bidirectional by definition, but zuluscsi never would drive it except as an initiator (which we don't do)"
Changed lines of the file:
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@@
   )
   (no_connect (at 124.46 55.88))
+  (no_connect (at 99.06 55.88))
   (no_connect (at 124.46 40.64))
+  (no_connect (at 99.06 40.64))
   (wire (pts (xy 247.65 38.1) (xy 247.65 40.64))
     (stroke (width 0) (type default))
@@
     (stroke (width 0) (type default))
   )
-  (wire (pts (xy 99.06 55.88) (xy 99.06 58.42))
-    (stroke (width 0) (type default))
-  )
   (wire (pts (xy 261.62 43.18) (xy 266.7 43.18))
     (stroke (width 0) (type default))
@@
     (stroke (width 0) (type default))
   )
-  (wire (pts (xy 93.98 36.83) (xy 99.06 40.64))
-    (stroke (width 0) (type default))
-  )
   (wire (pts (xy 247.65 74.93) (xy 247.65 77.47))
     (stroke (width 0) (type default))
@@
     (stroke (width 0) (type default))
   )
-  (wire (pts (xy 93.98 58.42) (xy 99.06 58.42))
-    (stroke (width 0) (type default))
-  )
   (wire (pts (xy 261.62 40.64) (xy 266.7 40.64))
     (stroke (width 0) (type default))
@@
     (effects (font (size 1.524 1.524)) (justify right bottom))
   )
-  (text "RST is input only in target mode.\nit is bidirectional by definition, \nbut zuluscsi never would drive it\nexcept as an initiator (which we don't do)"
-    (at 71.12 154.94 0)
+  (text "/RST is input only in target mode.\n\n/RST is bidirectional by definition, \nbut zuluscsi will not drive it in\ntarget mode, only as an initiator."
+    (at 69.85 156.21 0)
     (effects (font (size 1.524 1.524)) (justify left bottom))
   )
@@
     )
   )
-  (symbol (lib_id "zuluscsi-rescue:GND") (at 93.98 36.83 270) (unit 1)
-    (in_bom yes) (on_board yes) (dnp no)
-    (property "Reference" "#PWR046" (at 87.63 36.83 0)
-      (effects (font (size 1.27 1.27)) hide)
-    )
-    (property "Value" "GND" (at 88.9 36.83 90)
-      (effects (font (size 1.27 1.27)))
-    )
-    (property "Footprint" "" (at 93.98 36.83 0)
-      (effects (font (size 1.524 1.524)))
-    )
-    (property "Datasheet" "" (at 93.98 36.83 0)
-      (effects (font (size 1.524 1.524)))
-    )
-    (pin "1")
-    (instances
-      (project "SillyTinySCSI"
-        (path "/0a1a4d88-972a-46ce-b25e-6cb796bd41f7"
-          (reference "#PWR046") (unit 1)
-        )
-      )
-    )
-  )
   (symbol (lib_id "power:+2V8") (at 38.1 124.46 0) (unit 1)
     (in_bom yes) (on_board yes) (dnp no) (fields_autoplaced)
@@
         )
       )
-    )
-  )
-  (symbol (lib_id "zuluscsi-rescue:GND") (at 93.98 58.42 270) (unit 1)
-    (in_bom yes) (on_board yes) (dnp no)
-    (property "Reference" "#PWR045" (at 87.63 58.42 0)
-      (effects (font (size 1.27 1.27)) hide)
-    )
-    (property "Value" "GND" (at 88.9 58.42 90)
-      (effects (font (size 1.27 1.27)))
-    )
-    (property "Footprint" "" (at 93.98 58.42 0)
-      (effects (font (size 1.524 1.524)))
-    )
-    (property "Datasheet" "" (at 93.98 58.42 0)
-      (effects (font (size 1.524 1.524)))
-    )
-    (pin "1")
-    (instances
-      (project "SillyTinySCSI"
-        (path "/0a1a4d88-972a-46ce-b25e-6cb796bd41f7"
-          (reference "#PWR045") (unit 1)
-        )
-      )
