File: V2.0/cpu.kicad_sch (KiCad schematic)
At the start: 17 parts, among them J2 Micro_SD_Card_Det1, U1 74LVT125, U6 Pico W

Commit message: bring current
Other:
- note added: "Resistor settings correspond to DBGlog off, initator off, term on. DBGlog can be turned on in .ini file. GPIO ACK is pulled down to detect the PCB is not a Zulu Pico 2023b board at boot. The rev 2023b board has a broken DBGLOG and TERM_EN circuit."
- note added: "VBUS -> Diode -> VSYS on the RP2040 module Pico has plenty of onboard capacitance and will operate down to ~1.8v"
- note added: "resistor maintains compatibility with Zulu pico which may switch GP21 temporarily to output"
- note removed: "GPIO ACK is pulled down to detect the PCB is not a rev 2023b board at boot. The rev 2023b board has a broken DBGLOG and TERM_EN circuit. Static settings correspond to DBGlog off, initator off and term on"
- note removed: "VBUS -> Diode -> VSYS on the RP2040 module Pico has plenty of onboard capacitance"
- note removed: "resistor maintain HW compatibility with Zulu pico which may switch GP21 temporarily to output"
Changed lines of the file:
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@@
-    (stroke (width 0) (type default))
-  )
-  (wire (pts (xy 67.31 119.38) (xy 58.42 119.38))
     (stroke (width 0) (type default))
   )
@@
     (stroke (width 0) (type default))
   )
+  (wire (pts (xy 67.31 121.92) (xy 67.31 119.38))
+    (stroke (width 0) (type default))
+  )
   (wire (pts (xy 201.93 133.35) (xy 210.82 133.35))
     (stroke (width 0) (type default))
@@
     (stroke (width 0) (type default))
   )
-  (text "GPIO ACK is pulled down to \ndetect the PCB is not a rev 2023b\nboard at boot. The rev 2023b board\nhas a broken DBGLOG and TERM_EN\ncircuit.\n\nStatic settings correspond to \nDBGlog off, initator off\nand term on"
-    (at 186.69 55.88 0)
+  (text "Resistor settings correspond to \nDBGlog off, initator off, term on. \nDBGlog can be turned on in .ini file.\n\n\nGPIO ACK is pulled down to detect \nthe PCB is not a Zulu Pico 2023b\nboard at boot. The rev 2023b board\nhas a broken DBGLOG and TERM_EN\ncircuit.\n\n"
+    (at 186.69 63.5 0)
     (effects (font (size 1.524 1.524)) (justify left bottom))
   )
@@
     (effects (font (size 1.524 1.524)) (justify left bottom))
   )
-  (text "resistor maintain HW compatibility\nwith Zulu pico which may switch \nGP21 temporarily to output\n"
+  (text "resistor maintains compatibility\nwith Zulu pico which may switch \nGP21 temporarily to output\n"
     (at 140.97 62.23 0)
     (effects (font (size 1.524 1.524)) (justify left bottom))
   )
-  (text "VBUS -> Diode -> VSYS on the RP2040 module\nPico has plenty of onboard capacitance"
-    (at 111.76 31.75 0)
+  (text "VBUS -> Diode -> VSYS on the RP2040 module\nPico has plenty of onboard capacitance\nand will operate down to ~1.8v"
+    (at 110.49 30.48 0)
     (effects (font (size 1.524 1.524)) (justify left bottom))
   )
@@
     )
   )
-  (symbol (lib_id "zuluscsi-rescue:GND") (at 58.42 119.38 270) (mirror x) (unit 1)
-    (in_bom yes) (on_board yes) (dnp no)
-    (property "Reference" "#PWR02" (at 52.07 119.38 0)
-      (effects (font (size 1.27 1.27)) hide)
-    )
-    (property "Value" "GND" (at 55.1688 119.253 90)
+  (symbol (lib_id "zuluscsi-rescue:GND") (at 67.31 121.92 0) (mirror y) (unit 1)
+    (in_bom yes) (on_board yes) (dnp no)
+    (property "Reference" "#PWR02" (at 67.31 128.27 0)
+      (effects (font (size 1.27 1.27)) hide)
+    )
+    (property "Value" "GND" (at 64.77 125.73 0)
       (effects (font (size 1.27 1.27)) (justify right))
     )
-    (property "Footprint" "" (at 58.42 119.38 0)
-      (effects (font (size 1.27 1.27)) hide)
-    )
-    (property "Datasheet" "" (at 58.42 119.38 0)
-      (effects (font (size 1.27 1.27)) hide)
-    )
+    (property "Footprint" "" (at 67.31 121.92 0)
+      (effects (font (size 1.27 1.27)) hide)
+    )
+    (property "Datasheet" "" (at 67.31 121.92 0)
+      (effects (font (size 1.27 1.27)) hide)
+    )
